File: arduinouno.sch (KiCad schematic (older format))
At the start: 104 parts, among them J1 M20-7820842, J2 PAD_WITH_HOLE_4mmx1.5mm, J3 67997-106HLF, J4 67997-106HLF, J5 M20-7821046, J6 M20-7820646, J7 M20-7820842, J8 PAD_WITH_HOLE_4mmx1.5mm, SW1 1825910-6, SW2 1825910-6, U1 SN74AHC1G09DBVR, U2 SN74AHC1G09DBVR, U3 ATMEGA328P-PU, U4 ATMEGA16U2-AU, U5 SN74AHC1G09DBVR, U6 TL1963A-33DCQR, U7 10118193-0001LF, U8 SN74AHC1G09DBVR, Y1 16.000MHz, Y2 16.000MHz

Commit message: Schematic and README updates
Parts:
- added J7: 68602-104HLF, arduinouno:HDR_2x2_2.54mm, symbol arduinouno:68602-104HLF
- added JP1: 68000-103HLF, arduinouno:3P_Header_2.54mm, symbol arduinouno:68000-103HLF
- added LINK1: QPC02SXGN-RC, symbol arduinouno:QPC02SXGN-RC
- added R16: 0R, arduinouno:R0805x60mm, symbol arduinouno:RC0805JR-070RL
- SCKT_FOR_U1: renamed from SCKT1; value 4828-3004-CP -> 28-DIP Socket
- renumbered C4 to C1, C27 to C10, C3 to C13, C9 to C14, C13 to C17, C14 to C18, C10 to C19, C1 to C2, C29 to C20, C28 to C21, C17 to C22, C18 to C23, C19 to C24, C6 to C25, C20 to C26, C21 to C27, C22 to C28, C32 to C29, C5 to C3, C33 to C30, C24 to C31, C23 to C32, C25 to C33, C30 to C4, C7 to C5, C2 to C6, C8 to C7, C31 to C8, C26 to C9, D3 to D2, D4 to D3, D2 to D4, J8 to J3, J5 to J4, J6 to J5, J7 to J6, U7 to J7, J3 to J8, J4 to J9, JP1 to JP3, LINK1 to LINK2, LINK2 to LINK3, R5 to R10, R6 to R11, R8 to R12, R7 to R13, R9 to R14, R17 to R15, R18 to R17, R24 to R18, R11 to R20, R12 to R21, R13 to R22, R20 to R23, R25 to R24, R10 to R25, R14 to R27, R15 to R3, R21 to R4, R16 to R5, R22 to R6, R23 to R7, R3 to R8, R4 to R9, U3 to U1, U4 to U2, U1 to U2, U5 to U3, U6 to U4, U2 to U5
Connections:
- net labels added: 16U2_PB5, 16U2_PB7
- wire segments 361 -> 394
- no-connect marks 15 -> 12
Other:
- note added: "(c) 2015 Designed by FEDEVEL Academy http://www.fedevel.com/academy. Based on Arduino: http://www.arduino.cc. Released under Creative Commons Attribution-ShareAlike 3.0 Unported."
- note added: "16U2"
- note added: "28-PINS PROJECT"
- note added: "328P"
- note added: "3V3 LDO"
- note added: "AD"
- note added: "DESIGN NOTE:\nPin 8 (VIN) is not supported."
- note added: "DIP Socket"
- note added: "Design by FEDEVEL Academy"
- note added: "Differential Pair"
- note added: "Fiducials"
- note added: "Fiducials 4x Top"
- note added: "ICSP"
- note added: "ICSP1"
- note added: "IOH"
- note added: "IOL"
- note added: "Implemented by Phil McMillan in"
- note added: "JP1"
- note added: "JP2"
- note added: "JP3"
- note added: "Micro USB"
- note added: "Mounting Holes"
- note added: "Mounting Holes (7.4mm pad, 3.2mm drill)\nBOARD MOUNTING HOLES - ONE IN EACH CORNER"
- note added: "NP"
- note added: "Power"
- note added: "Power LED"
- note added: "Power Pads"
- note added: "Power Selection"
- note added: "Power flags for design rules check.\n"
- note added: "Reset (16U2)"
- note added: "Reset (328P)"
- note added: "This means you can use it on your own derived works, in part or completely, as long as you also adopt the same licence. You find the complete text of the licence here.: http://creativecommons.org/licenses/by-sa/3.0/legalcode"
- note added: "User Button"
- note added: "User LED"

Commit message: Completed schematic capture
Parts:
- renumbered C4 to C1, C16 to C10, C31 to C11, C10 to C12, C21 to C13, C1 to C14, C3 to C15, C5 to C16, C33 to C17, C17 to C19, C8 to C2, C23 to C20, C28 to C21, C18 to C22, C24 to C23, C26 to C24, C11 to C25, C9 to C26, C12 to C27, C25 to C28, C30 to C29, C14 to C3, C6 to C30, C2 to C31, C13 to C32, C29 to C33, C7 to C34, C19 to C4, C22 to C5, C27 to C6, C20 to C7, C32 to C8, C15 to C9, D2 to D1, D3 to D2, D5 to D3, D6 to D4, D1 to D5, D4 to D6, J5 to J2, J6 to J3, J9 to J5, J8 to J6, J2 to J8, J3 to J9, JP3 to JP1, J7 to JP2, JP2 to JP3, JP1 to JP4, LINK2 to LINK1, LINK3 to LINK2, LINK1 to LINK3, R17 to R1, R21 to R10, R22 to R11, R27 to R12, R20 to R13, R11 to R14, R5 to R15, R12 to R16, R3 to R17, R10 to R18, R1 to R19, R19 to R2, R8 to R20, R18 to R21, R26 to R22, R2 to R23, R9 to R24, R24 to R25, R15 to R27, R16 to R28, R23 to R3, R13 to R4, R25 to R5, R4 to R8, R14 to R9, U4 to U3, U3 to U4, U2 to U5, U5 to U6, U8 to U7
Connections:
- net labels added: 16U2_PB6
Other:
- note added: "= Not Fitted"
- note added: "DESIGN NOTE: \n\nAbout JP1:\n1) Autoreset Enabled - Short 1&2. Int his case, 16U2 is used to reset 328P when\nfirmware inside 328P is updated from Arduino IDE.\n\n2) 16U2 DFU mode enabled - Short 2&3. 16U2 HWB pin is sampled by 16U2 during\nRESET. If pulled low, then after Reset the 16U2 will go into DFU mode (it’s the mode\nwhere you can flash 16U2 firmware through USB and Atmel Flip software.\n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"
- note added: "DESIGN NOTE:\nThis LED is inverted.\n- SCK High = LED OFF\n- SCK Low = LED ON"
- note added: "DESIGN NOTE:\nThis board can be powered from micro USB\nconnector (J7) or a single +3.3V power rail\n(through J1 pin 4). If +3.3V is used, fit R26\nand R28. In this case, JP4 and R27 must NOT be\nfitted, otherwise the board may be damaged."
- note added: "DESIGN NOTE:\nThis board supports 5V or 3V3 voltage level on the IO pins.\n1) 5V IO - Fit everything as defined in this schematic. NF means do not fit this component.\n\n2) 3.3V IO - Remove R27, Fit R28, * Replace Y1 (change from 16MHz to 10MHz), * Replace Y2\n(change from 16MHz to 8MHz).\n\n3) Both 5V and 3V3, selected through JP4 - Remove R27, Remove R28, Fit JP4, * Replace Y1\n(change from 16M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"
- note added: "DESIGN NOTE:\n\nAbout JP3:\n1) DebugWire support - Short 1&2. This was added to support possible debugWire debugging\n(programming?) of 328P through 16U2. In this case, the 16U2 needs to have a correct\nfirmware and has to behave as a debugWire tool.\n\n2) ISP programmer mode - Short 2&3. In this case, take a cable and connect J5 and J6\ntogether. Upload AVRISP MkII firmware in the 16U2 and you c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"
- note added: "Key"
- note added: "LAYOUT NOTE:\n1) Route all the POWER tracks with minimum track width 0.4mm.\n2) Route all the other tracks by 0.4mm and change them by the end of\nthe design to 0.2mm."
- note added: "NF"
- note removed: "NP"

Commit message: Added schematic pdf, updated missing R26
Parts:
- added R26: 0R, arduinouno:R0805x60mm, symbol arduinouno:RC0805JR-070RL
Connections:
- wire segments 394 -> 398
Changed lines of the file:
@@
 L arduinouno:MPZ2012S601AT000 FB1
 U 1 1 5B98354B
-P 8000 3500
-F 0 "FB1" H 8000 3600 50  0000 C CNN
-F 1 "MPZ2012S601AT000" H 8000 3400 50  0001 C CNN
-F 2 "arduinouno:FB0805x85mm" H 8000 3100 50  0001 C CNN
-F 3 "https://product.tdk.com/info/en/catalog/datasheets/beads_commercial_power_mpz2012_en.pdf" H 8050 3300 50  0001 C CNN
-F 4 "445-7645-1-ND" H 8000 3200 50  0001 C CNN "Digikey"
-	1    8000 3500
+P 7500 3500
+F 0 "FB1" H 7500 3600 50  0000 C CNN
+F 1 "MPZ2012S601AT000" H 7500 3400 50  0001 C CNN
+F 2 "arduinouno:FB0805x85mm" H 7500 3100 50  0001 C CNN
+F 3 "https://product.tdk.com/info/en/catalog/datasheets/beads_commercial_power_mpz2012_en.pdf" H 7550 3300 50  0001 C CNN
+F 4 "445-7645-1-ND" H 7500 3200 50  0001 C CNN "Digikey"
+	1    7500 3500
 	1    0    0    -1
 $EndComp
@@
 L arduinouno:C2012X5R1C106M085AC C3
 U 1 1 5B9839B3
-P 8300 3700
-F 0 "C3" V 8200 3700 50  0000 L CNN
-F 1 "10uF|16V" V 8400 3700 50  0000 L CNN
-F 2 "arduinouno:C0805x145mm" H 8300 3250 50  0001 C CNN
-F 3 "https://product.tdk.com/info/en/catalog/datasheets/mlcc_commercial_general_en.pdf" H 8450 3450 50  0001 C CNN
-F 4 "445-7645-1-ND" H 8300 3350 50  0001 C CNN "Digikey"
-	1    8300 3700
+P 7800 3700
+F 0 "C3" V 7700 3700 50  0000 L CNN
+F 1 "10uF|16V" V 7900 3700 50  0000 L CNN
+F 2 "arduinouno:C0805x145mm" H 7800 3250 50  0001 C CNN
+F 3 "https://product.tdk.com/info/en/catalog/datasheets/mlcc_commercial_general_en.pdf" H 7950 3450 50  0001 C CNN
+F 4 "445-7645-1-ND" H 7800 3350 50  0001 C CNN "Digikey"
+	1    7800 3700
 	0    1    1    0
 $EndComp
@@
 L arduinouno:C2012X7R1H104K085AA C4
 U 1 1 5B983BC3
-P 8800 3700
-F 0 "C4" V 8700 3700 50  0000 L CNN
-F 1 "100nF" V 8900 3700 50  0000 L CNN
-F 2 "arduinouno:C0805x95mm" H 8800 3250 50  0001 C CNN
-F 3 "https://product.tdk.com/info/en/catalog/datasheets/mlcc_commercial_general_en.pdf" H 8950 3450 50  0001 C CNN
-F 4 "445-7534-1-ND" H 8800 3350 50  0001 C CNN "Digikey"
-	1    8800 3700
+P 8300 3700
+F 0 "C4" V 8200 3700 50  0000 L CNN
+F 1 "100nF" V 8400 3700 50  0000 L CNN
+F 2 "arduinouno:C0805x95mm" H 8300 3250 50  0001 C CNN
+F 3 "https://product.tdk.com/info/en/catalog/datasheets/mlcc_commercial_general_en.pdf" H 8450 3450 50  0001 C CNN
+F 4 "445-7534-1-ND" H 8300 3350 50  0001 C CNN "Digikey"
+	1    8300 3700
 	0    1    1    0
 $EndComp
@@
 L arduinouno:C2012X7R1H104K085AA C5
 U 1 1 5B983D68
-P 9200 3700
-F 0 "C5" V 9100 3700 50  0000 L CNN
-F 1 "100nF" V 9300 3700 50  0000 L CNN
-F 2 "arduinouno:C0805x95mm" H 9200 3250 50  0001 C CNN
-F 3 "https://product.tdk.com/info/en/catalog/datasheets/mlcc_commercial_general_en.pdf" H 9350 3450 50  0001 C CNN
-F 4 "445-7534-1-ND" H 9200 3350 50  0001 C CNN "Digikey"
-	1    9200 3700
+P 8700 3700
+F 0 "C5" V 8600 3700 50  0000 L CNN
+F 1 "100nF" V 8800 3700 50  0000 L CNN
+F 2 "arduinouno:C0805x95mm" H 8700 3250 50  0001 C CNN
+F 3 "https://product.tdk.com/info/en/catalog/datasheets/mlcc_commercial_general_en.pdf" H 8850 3450 50  0001 C CNN
+F 4 "445-7534-1-ND" H 8700 3350 50  0001 C CNN "Digikey"
+	1    8700 3700
 	0    1    1    0
 $EndComp
@@
 L arduinouno:GND #PWR054
 U 1 1 5B99258B
-P 9200 3850
-F 0 "#PWR054" H 9200 3600 50  0001 C CNN
-F 1 "GND" H 9200 3700 50  0001 C CNN
-F 2 "" H 9200 3850 50  0001 C CNN
-F 3 "" H 9200 3850 50  0001 C CNN
-	1    9200 3850
+P 8700 3850
+F 0 "#PWR054" H 8700 3600 50  0001 C CNN
+F 1 "GND" H 8700 3700 50  0001 C CNN
+F 2 "" H 8700 3850 50  0001 C CNN
+F 3 "" H 8700 3850 50  0001 C CNN
+	1    8700 3850
 	1    0    0    -1
 $EndComp
@@
 L arduinouno:GND #PWR050
 U 1 1 5B9925D2
-P 8800 3850
-F 0 "#PWR050" H 8800 3600 50  0001 C CNN
-F 1 "GND" H 8800 3700 50  0001 C CNN
-F 2 "" H 8800 3850 50  0001 C CNN
-F 3 "" H 8800 3850 50  0001 C CNN
-	1    8800 3850
-	1    0    0    -1
-$EndComp
-$Comp
-L arduinouno:GND #PWR046
-U 1 1 5B992619
 P 8300 3850
-F 0 "#PWR046" H 8300 3600 50  0001 C CNN
+F 0 "#PWR050" H 8300 3600 50  0001 C CNN
 F 1 "GND" H 8300 3700 50  0001 C CNN
 F 2 "" H 8300 3850 50  0001 C CNN
@@
 $EndComp
 $Comp
+L arduinouno:GND #PWR046
+U 1 1 5B992619
+P 7800 3850
+F 0 "#PWR046" H 7800 3600 50  0001 C CNN
+F 1 "GND" H 7800 3700 50  0001 C CNN
+F 2 "" H 7800 3850 50  0001 C CNN
+F 3 "" H 7800 3850 50  0001 C CNN
+	1    7800 3850
+	1    0    0    -1
+$EndComp
+$Comp
 L arduinouno:+5V_3V3 #PWR038
 U 1 1 5B992E59
-P 7700 3500
-F 0 "#PWR038" H 7700 3200 50  0001 C CNN
-F 1 "+5V_3V3" H 7700 3650 50  0000 C CNN
-F 2 "" H 7700 3500 50  0001 C CNN
-F 3 "" H 7700 3500 50  0001 C CNN
-	1    7700 3500
+P 7200 3500
+F 0 "#PWR038" H 7200 3200 50  0001 C CNN
+F 1 "+5V_3V3" H 7200 3650 50  0000 C CNN
+F 2 "" H 7200 3500 50  0001 C CNN
+F 3 "" H 7200 3500 50  0001 C CNN
+	1    7200 3500
 	1    0    0    -1
 $EndComp
 Wire Wire Line
-	7700 3500 7800 3500
+	7200 3500 7300 3500
 $Comp
 L arduinouno:+5V_3V3 #PWR041
@@
 $EndComp
 Wire Wire Line
-	8200 3500 8300 3500
+	7700 3500 7800 3500
 Wire Wire Line
-	8300 3550 8300 3500
-Connection ~ 8300 3500
+	7800 3550 7800 3500
+Connection ~ 7800 3500
 Wire Wire Line
-	8300 3500 8800 3500
+	7800 3500 8300 3500
 Wire Wire Line
-	8800 3550 8800 3500
-Connection ~ 8800 3500
+	8300 3550 8300 3500
+Connection ~ 8300 3500
 Wire Wire Line
-	8800 3500 9200 3500
+	8300 3500 8700 3500
 Wire Wire Line
-	9200 3550 9200 3500
-Connection ~ 9200 3500
+	8700 3550 8700 3500
+Connection ~ 8700 3500
 Wire Wire Line
-	9200 3500 10300 3500
+	8700 3500 9500 3500
 Wire Wire Line
 	10000 3950 10000 3900
@@
 	3200 14750 3300 14750
 Wire Wire Line
-	10300 4400 9650 4400
+	10300 4400 9150 4400
 $Comp
 L arduinouno:RC0805FR-0710KL R4
 U 1 1 5BD57A80
-P 9650 4150
-F 0 "R4" V 9604 4228 50  0000 L CNN
-F 1 "10k" V 9695 4228 50  0000 L CNN
-F 2 "arduinouno:R0805x60mm" H 9650 3750 50  0001 C CNN
-F 3 "http://www.yageo.com/documents/recent/PYu-RC_Group_51_RoHS_L_9.pdf" H 9600 3950 50  0001 C CNN
-F 4 "311-10.0KCRCT-ND" H 9650 3850 50  0001 C CNN "Digikey"
-	1    9650 4150
+P 9150 4150
+F 0 "R4" V 9104 4228 50  0000 L CNN
+F 1 "10k" V 9195 4228 50  0000 L CNN
+F 2 "arduinouno:R0805x60mm" H 9150 3750 50  0001 C CNN
+F 3 "http://www.yageo.com/documents/recent/PYu-RC_Group_51_RoHS_L_9.pdf" H 9100 3950 50  0001 C CNN
+F 4 "311-10.0KCRCT-ND" H 9150 3850 50  0001 C CNN "Digikey"
+	1    9150 4150
 	0    1    1    0
 $EndComp
-Connection ~ 9650 4400
+Connection ~ 9150 4400
 Wire Wire Line
-	9650 4400 9050 4400
-Text Label 9050 4400 0    50   ~ 0
+	9150 4400 8450 4400
+Text Label 8450 4400 0    50   ~ 0
 16U2_RESETn
 $Comp
 L arduinouno:+5V_3V3 #PWR060
 U 1 1 5BDFC1A8
-P 9650 3900
-F 0 "#PWR060" H 9650 3600 50  0001 C CNN
-F 1 "+5V_3V3" H 9650 4050 50  0000 C CNN
-F 2 "" H 9650 3900 50  0001 C CNN
-F 3 "" H 9650 3900 50  0001 C CNN
-	1    9650 3900
+P 9150 3900
+F 0 "#PWR060" H 9150 3600 50  0001 C CNN
+F 1 "+5V_3V3" H 9150 4050 50  0000 C CNN
+F 2 "" H 9150 3900 50  0001 C CNN
+F 3 "" H 9150 3900 50  0001 C CNN
+	1    9150 3900
 	1    0    0    -1
 $EndComp
@@
 L arduinouno:C2012X5R1E105K125AA C7
 U 1 1 5C4CBD49
-P 9000 4600
-F 0 "C7" H 8850 4650 50  0000 C CNN
-F 1 "1uF|25V" H 9250 4650 50  0000 C CNN
-F 2 "arduinouno:C0805x95mm" H 9000 4150 50  0001 C CNN
-F 3 "https://product.tdk.com/info/en/catalog/datasheets/mlcc_commercial_general_en.pdf" H 9150 4350 50  0001 C CNN
-F 4 "445-1419-1-ND" H 9000 4250 50  0001 C CNN "Digikey"
-	1    9000 4600
+P 8800 4600
+F 0 "C7" H 8650 4650 50  0000 C CNN
+F 1 "1uF|25V" H 9050 4650 50  0000 C CNN
+F 2 "arduinouno:C0805x95mm" H 8800 4150 50  0001 C CNN
+F 3 "https://product.tdk.com/info/en/catalog/datasheets/mlcc_commercial_general_en.pdf" H 8950 4350 50  0001 C CNN
+F 4 "445-1419-1-ND" H 8800 4250 50  0001 C CNN "Digikey"
+	1    8800 4600
 	1    0    0    -1
 $EndComp
 Wire Wire Line
-	9150 4600 10300 4600
+	8950 4600 9500 4600
 Wire Wire Line
-	8850 4600 8700 4600
+	8650 4600 8500 4600
 Text Label 9600 4600 0    50   ~ 0
 +3V3_16U2_UCAP
@@
 L arduinouno:GND #PWR049
 U 1 1 5C5633A9
-P 8700 4600
-F 0 "#PWR049" H 8700 4350 50  0001 C CNN
-F 1 "GND" H 8700 4450 50  0001 C CNN
-F 2 "" H 8700 4600 50  0001 C CNN
-F 3 "" H 8700 4600 50  0001 C CNN
-	1    8700 4600
+P 8500 4600
+F 0 "#PWR049" H 8500 4350 50  0001 C CNN
+F 1 "GND" H 8500 4450 50  0001 C CNN
+F 2 "" H 8500 4600 50  0001 C CNN
+F 3 "" H 8500 4600 50  0001 C CNN
+	1    8500 4600
 	1    0    0    -1
 $EndComp
@@
 Data
 89 50 4E 47 0D 0A 1A 0A 00 00 00 0D 49 48 44 52 00 00 01 24 00 00 00 AC 08 02 00 00 00 5D 0F 46
-BA 00 00 00 03 73 42 49 54 08 08 08 DB E1 4F E0 00 00 00 09 70 48 59 73 00 00 16 25 00 00 16 25
-01 49 52 24 F0 00 00 20 00 49 44 41 54 78 9C EC BD 57 93 5C 47 D2 25 78 DC E3 8A 54 A5 05 34 40
+BA 00 00 00 03 73 42 49 54 08 08 08 DB E1 4F E0 00 00 00 09 70 48 59 73 00 00 15 E0 00 00 15 E0
+01 8D 54 2C 38 00 00 20 00 49 44 41 54 78 9C EC BD 57 93 5C 47 D2 25 78 DC E3 8A 54 A5 05 34 40
 02 04 D9 24 9B EC EE F9 C4 7C 36 6B B6 66 F3 B2 FF 77 6D DF F6 61 F6 65 77 66 76 5A 51 80 D0 1A
 28 5D 95 5A DD 7B 23 DC E7 21 E2 DE CC 2A 80 DD 1F 41 B2 C0 E6 E4 31 20 AD 2A 2B C5 15 E1 E1 1E
@@
 Wire Notes Line
 	18100 5550 18100 4400
+$Comp
+L arduinouno:RC0805JR-070RL R26
+U 1 1 5DB354B8
+P 9500 3950
+F 0 "R26" H 9250 4000 50  0000 C CNN
+F 1 "0R" H 9700 4000 50  0000 C CNN
+F 2 "arduinouno:R0805x60mm" H 9500 3550 50  0001 C CNN
+F 3 "http://www.yageo.com/documents/recent/PYu-RC_Group_51_RoHS_L_9.pdf" H 9450 3750 50  0001 C CNN
+F 4 "311-0.0ARCT-ND" H 9500 3650 50  0001 C CNN "Digikey"
+	1    9500 3950
+	0    1    1    0
+$EndComp
+Wire Wire Line
+	9500 4200 9500 4600
+Connection ~ 9500 4600
+Wire Wire Line
+	9500 4600 10300 4600
+Wire Wire Line
+	9500 3700 9500 3500
+Connection ~ 9500 3500
+Wire Wire Line
+	9500 3500 10300 3500
+Text Notes 9350 4050 0    138  ~ 28
+NF
 $EndSCHEMATC
