File: arduinouno.kicad_pcb (KiCad board)
At the start: 2 copper layers, 68.6 x 53.3 mm, 107 parts, among them J1 M20-7820842, J2 M20-7820646, J3 M20-7820842, J4 M20-7821046, J5 67997-106HLF, J6 67997-106HLF, J7 10118193-0001LF, J8 PAD_WITH_HOLE_4mmx1.5mm, J9 PAD_WITH_HOLE_4mmx1.5mm, SW1 1825910-6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

Commit message: Updated pcb layout to Kicad 7.0
Other:
- net class Default removed
- net class Power removed
